File: hardware/hardware.sch (KiCad schematic (older format))
At the start: 14 parts, among them J1 VGA, U14 74LS273, X1 20MHz

Commit message: Clean up EEPROM framebuffer design
Drop the extra pins
Connections:
- net framebuffer/B0 renamed eeprom-framebuffer/B0
- net framebuffer/B1 renamed eeprom-framebuffer/B1
- net framebuffer/CLK renamed hsync/CLK
- net framebuffer/G0 renamed eeprom-framebuffer/G0
- net framebuffer/G1 renamed eeprom-framebuffer/G1
- net framebuffer/G2 renamed eeprom-framebuffer/G2
- net framebuffer/R0 renamed eeprom-framebuffer/R0
- net framebuffer/R1 renamed eeprom-framebuffer/R1
- net framebuffer/R2 renamed eeprom-framebuffer/R2
- no-connect marks 5 -> 6

Commit message: Drop another chip by stretching the vsync pulse
Works fine on my test LCDs.  No idea what would happen with a CRT.
Connections:
- no-connect marks 6 -> 5
Changed lines of the file:
@@
 F11 "Q0" O R 3000 4100 50
 F12 "VSYNC" O R 3000 3800 50
-F13 "~EOF~" O L 2400 4900 50
 $EndSheet
 Wire Wire Line
@@
 Wire Wire Line
 	8650 3000 8550 3000
-NoConn ~ 2400 4900
 Wire Wire Line
 	2200 5450 5650 5450
