File: hardware/hsync.sch (KiCad schematic (older format))
At the start: 6 parts, among them U1 74LS161, U2 74LS161, U3 74LS161, U4 74LS20, U5 74LS20, U6 74LS00

Commit message: Drop another chip by stretching the vsync pulse
Works fine on my test LCDs.  No idea what would happen with a CRT.
Changed lines of the file:
@@
 	6400 2250 6450 2250
-Wire Wire Line
-	6600 2250 6600 3200
-Connection ~ 6450 2250
-Wire Wire Line
-	6450 2250 6600 2250
 Wire Wire Line
 	5800 2350 5750 2350
@@
 Wire Wire Line
 	5450 2250 5450 2150
+Wire Wire Line
+	6450 2850 6600 2850
+Wire Wire Line
+	6600 2850 6600 3200
+Connection ~ 6450 2850
 $EndSCHEMATC
