File: hardware/vsync.sch (KiCad schematic (older format))
At the start: 6 parts, among them U10 74LS20, U11 74LS20, U12 74LS00, U7 74LS161, U8 74LS161, U9 74LS161

Commit message: Drop another chip by stretching the vsync pulse
Works fine on my test LCDs.  No idea what would happen with a CRT.
Parts:
- removed unit 3 of U10
- removed unit 1 of U11
- U9: renamed from U10; value 74LS20 -> 74LS10; symbol 74xx:74LS20 -> 74xx:74LS10
- U9: renamed from U11; value 74LS20 -> 74LS10
- U9: renamed from U11; value 74LS20 -> 74LS10; symbol 74xx:74LS20 -> 74xx:74LS10
- renumbered U12 to U10, U7 to U6, U8 to U7, U9 to U8
Connections:
- net labels removed: ~EOF~
- wire segments 157 -> 137
Other:
- moved on the sheet: U10C
